File: big_muff/big_muff.kicad_sch (KiCad schematic)
At the start: 51 parts, among them J1 PJ-202A, J3 Conn_01x04_Socket, Q1 2N5088, Q2 2N5088, Q3 2N5088, Q4 2N5088

Commit message: Continue work with big muff
Parts:
- removed Q1, Q2, Q3, Q4: 2N5088, 2N5088:TO92, symbol 2N5088:2N5088
- added D7: 1N4148, Diode_THT:D_DO-35_SOD27_P7.62mm_Horizontal, symbol Diode:1N4148
- added Q1, Q2, Q3, Q4: BC550, Package_TO_SOT_THT:TO-92_Inline, symbol Transistor_BJT:BC550
- C1, C10, C11, C12, C13, C2, C3, C4, C5, C6, C7, C8, C9: footprint Capacitor_THT:C_Axial_L5.1mm_D3.1mm_P7.50mm_Horizontal -> Capacitor_THT:C_Disc_D3.0mm_W2.0mm_P2.50mm
- C14: value 0.1u -> 1u; footprint Capacitor_THT:C_Axial_L5.1mm_D3.1mm_P7.50mm_Horizontal -> Capacitor_THT:C_Disc_D3.0mm_W2.0mm_P2.50mm
- R2: value 100k -> 47k
Connections:
- net +9V: now also D7.1 (K); no longer J1.1
- net GND: now also J1.1; no longer J1.2, J1.3
- net at C9.1, D3.1 (K), D4.2 (A)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: now also Q3.2 (B)
- net at C2.2, C3.1, R1.1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: now also Q1.1 (C)
- net at C1.2, C2.1, R1.2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: now also Q1.2 (B)
- net at C5.1, C6.1, R11.2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: now also Q2.2 (B)
- net at C10.1, C8.2, C9.2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: now also Q3.1 (C)
- net at C13.1, R24.2: now also Q4.1 (C)
- net at C5.2, C7.1, D1.2 (A)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: now also Q2.1 (C)
- net at C12.2, R21.1, R23.2: now also Q4.2 (B)
- net at R22.1: now also Q4.3 (E)
- net at R3.1: now also Q1.3 (E)
- net at R17.2: now also Q3.3 (E)
- net at R12.2: now also Q2.3 (E)
- new net: D7.2 (A), J1.2, J1.3
- no-connect marks 0 -> 1
Other:
- moved on the sheet: C6
